Commit message: Cleaned up the hopping_robot's gym environment. I also added more information to the state vectors. There should be velocity info in the observation vectors

File: DDPG/h3pper/gym-hopping_robot/gym_hopping_robot/envs/hopping_robot/urdf/hopping_robot.urdf (robot description, URDF)
Before this commit: robot hopping_robot, 5 links, 4 joints
Joints:
- joint leg_foot: limit lower=0.0 upper=1.57 effort=10 velocity=1.0 -> lower=-1.57 upper=1.57 effort=10 velocity=1.0

File: DDPG/h3pper/gym-hopping_robot/gym_hopping_robot/envs/hopping_robot/urdf/hopping_robot.xacro (robot description, xacro)
@@ -126,8 +126,8 @@
                                 <!-- color rgba="0 255 0 0.5" / -->
                         </material>
-			<origin rpy="0 0 0" xyz="0.0 ${-foot_height/2} 0.0"/>
+			<origin rpy="0 0 0" xyz="0.0 0.0 0.0"/>
                 </visual>
                 <inertial>
-			<origin rpy="0 0 0" xyz="0.0 ${-foot_height/2} 0.0"/>
+			<origin rpy="0 0 0" xyz="0.0 0.0 0.0"/>
                         <mass value = "1.0"/>
                         <!-- Fix the inertia tag-->
@@ -137,5 +137,5 @@
                 </inertial>
                 <collision>
-			<origin rpy="0 0 0" xyz="0.0 ${-foot_height/2} 0.0"/>
+			<origin rpy="0 0 0" xyz="0.0 0.0 0.0"/>
                         <geometry>
                                 <box size="${foot_width} ${foot_height} ${foot_depth}" />
@@ -171,5 +171,5 @@
 		<child link="foot" />
 		<!-- What to set these to? -->
-	  	<limit velocity="1.0" effort="10" lower="0.0" upper="1.57"/>
+	  	<limit velocity="1.0" effort="10" lower="-1.57" upper="1.57"/>
   	</joint>
 	 <transmission name="leg_foot_trans" type="transmission_interface/SimpleTransmission">
