Commit message: I integrated Dan's optimal controller trajectory generator into the PMTG architecture gym environment. I ran it for about 10 minutes and it did not seem to learn anything (yet)

File: PMTG/gym-hopping_robot_pmtg/gym_hopping_robot_pmtg/envs/urdf/hopping_robot.urdf (robot description, URDF)
Before this commit: robot hopping_robot, 5 links, 4 joints
Joints:
- joint leg_foot: limit lower=-1.57 upper=1.57 effort=10 velocity=1.0 -> lower=-0.785 upper=0.785 effort=10 velocity=1.0
- joint link1_link2: limit lower=-1.57 upper=1.57 effort=10 velocity=1.0 -> lower=-0.785 upper=0.785 effort=10 velocity=1.0
- joint link2_link3: limit lower=-1.57 upper=1.57 effort=10 velocity=1.0 -> lower=-0.785 upper=0.785 effort=10 velocity=1.0

File: PMTG/gym-hopping_robot_pmtg/gym_hopping_robot_pmtg/envs/urdf/hopping_robot.xacro (robot description, xacro)
@@ -155,5 +155,5 @@
                 <child link="link2" />
                 <!-- What to set these to? -->
-                <limit velocity="1.0" effort="10" lower="-1.57" upper="1.57"/>
+		<limit velocity="1.0" effort="10" lower="${-1.57/2.0}" upper="${1.57/2.0}"/>
 	</joint>
 	<joint name="link2_link3" type="revolute">
@@ -163,5 +163,5 @@
                 <child link="link3" />
                 <!-- What to set these to? -->
-                <limit velocity="1.0" effort="10" lower="-1.57" upper="1.57"/>
+		<limit velocity="1.0" effort="10" lower="${-1.57/2.0}" upper="${1.57/2.0}"/>
         </joint>
 	<joint name="leg_foot" type="revolute">
@@ -171,5 +171,5 @@
 		<child link="foot" />
 		<!-- What to set these to? -->
-	  	<limit velocity="1.0" effort="10" lower="-1.57" upper="1.57"/>
+		<limit velocity="1.0" effort="10" lower="${-1.57/2.0}" upper="${1.57/2.0}"/>
   	</joint>
 	 <transmission name="leg_foot_trans" type="transmission_interface/SimpleTransmission">
